Commit message: zmodyfikowany: lab2/models/move.urdf

File: lab2/models/move.urdf (robot description, URDF)
Before this commit: robot robot, 4 links, 3 joints
Joints:
- joint base_to_link1: limit lower=-3.1415 upper=3.1415 effort=1000.0 velocity=0.5 -> lower=-0.2 upper=0 effort=1000.0 velocity=0.5; type revolute -> prismatic
- joint link1_to_link2: limit lower=-1.57075 upper=1.57075 effort=1000.0 velocity=0.5 -> lower=-0.2 upper=0 effort=1000.0 velocity=0.5; type revolute -> prismatic
