Commit message: zmodyfikowany: lab_4/launch/rviz.launch 	zmodyfikowany: lab_4/models/move.urdf 	nowy plik:     lab_4/pictures/10.png 	nowy plik:     lab_4/pictures/7.png 	nowy plik:     lab_4/pictures/8.png 	nowy plik:     lab_4/pictures/9.png 	nowy plik:     lab_4/rviz/urdf.rviz 	zmodyfikowany: lab_4/scripts/jint.py

File: lab_4/models/move.urdf (robot description, URDF)
Before this commit: robot robot, 4 links, 3 joints
Joints:
- joint link1_to_link2: limit lower=-0.2 upper=0.1 effort=1000.0 velocity=0.5 -> lower=-0.2 upper=0 effort=1000.0 velocity=0.5
